Commit message: include updated xacro

File: land_description/urdf/land_description.urdf.xacro (robot description, xacro)
@@ -223,5 +223,5 @@
     <parent link="base_link"/>
     <child link="lidar_link"/>
-    <origin rpy="0 0 0" xyz="0 0 0.1055"/>
+    <origin rpy="0 0 3.14159" xyz="0 0 0.1055"/>
   </joint>
   <!-- CAMERA -->

Commit message: test update to urdf

File: land_description/urdf/land_description.urdf.xacro (robot description, xacro)
@@ -200,5 +200,5 @@
     <parent link="base_link"/>
     <child link="imu_link"/>
-    <origin rpy="0 0 0" xyz="0.04 0 0.0305"/>
+    <origin rpy="0 0 1.5707963267948966" xyz="0.04 0 0.0305"/>
   </joint>
   <!-- LIDAR -->
