Commit message: further work on ros2_control

File: land_description/urdf/land_description.urdf (robot description, URDF)
Before this commit: robot land, 3 links, 2 joints
Links:
- added link imu_link; collision box size=0.02 0.01 0.001; visual box size=0.02 0.01 0.001
- added link lidar_link; collision cylinder length=0.018 radius=${0.051/2}; visual cylinder length=0.018 radius=${0.051/2}
Joints:
- added joint imu_joint: type fixed, parent base_link, child imu_link, origin xyz=${0.01+tower_length/2} 0 ${base_height/2} rpy=0 0 0
- added joint lidar_joint: type fixed, parent base_link, child lidar_link, origin xyz=0 0 ${base_height/2 + tower_height/2 + 0.018/2} rpy=0 0 0

Commit message: test hardware camera node

File: land_description/urdf/land_description.urdf (robot description, URDF)
Before this commit: robot land, 5 links, 4 joints
Links:
- added link camera_link; collision box size=0.001 0.025 0.025; visual box size=0.001 0.025 0.025
Joints:
- added joint camera_joint: type fixed, parent base_link, child camera_link, origin xyz=${tower_length/2} 0 ${base_height/2 + (3*tower_height/4)} rpy=0 0 0

File: land_description/urdf/land_description.urdf.xacro (robot description, xacro)
@@ -225,4 +225,27 @@
     <origin rpy="0 0 0" xyz="0 0 0.0725"/>
   </joint>
+  <!-- CAMERA -->
+  <link name="camera_link">
+    <visual name="camera_link_visual">
+      <geometry>
+        <box size="0.001 0.025 0.025"/>
+      </geometry>
+    </visual>
+    <collision name="camera_link_collision">
+      <geometry>
+        <box size="0.001 0.025 0.025"/>
+      </geometry>
+    </collision>
+    <inertial>
+      <origin rpy="1.5707963267948966 0 1.5707963267948966" xyz="0 0 0"/>
+      <mass value="0.01"/>
+      <inertia ixx="5.216666666666668e-07" ixy="0.0" ixz="0.0" iyy="5.216666666666668e-07" iyz="0.0" izz="1.041666666666667e-06"/>
+    </inertial>
+  </link>
+  <joint name="camera_joint" type="fixed">
+    <parent link="base_link"/>
+    <child link="camera_link"/>
+    <origin rpy="0 0 0" xyz="0.03 0 0.08"/>
+  </joint>
   <!-- ROS2 WHEEL CONTROL -->
   <ros2_control name="MecanumHardware" type="system">

Commit message: fix for lidar urdf height

File: land_description/urdf/land_description.urdf (robot description, URDF)
Before this commit: robot land, 6 links, 5 joints
Joints:
- joint lidar_joint: origin xyz=0 0 ${base_height/2 + tower_height/2 + 0.018/2} rpy=0 0 0 -> xyz=0 0 ${base_height/2 + tower_height + 0.018/2} rpy=0 0 0

File: land_description/urdf/land_description.urdf.xacro (robot description, xacro)
@@ -223,5 +223,5 @@
     <parent link="base_link"/>
     <child link="lidar_link"/>
-    <origin rpy="0 0 0" xyz="0 0 0.0725"/>
+    <origin rpy="0 0 0" xyz="0 0 0.1055"/>
   </joint>
   <!-- CAMERA -->

Commit message: rotated lidar urdf

File: land_description/urdf/land_description.urdf (robot description, URDF)
Before this commit: robot land, 6 links, 5 joints
Joints:
- joint lidar_joint: origin xyz=0 0 ${base_height/2 + tower_height + 0.018/2} rpy=0 0 0 -> xyz=0 0 ${base_height/2 + tower_height + 0.018/2} rpy=0 0 3.14159

Commit message: update urdf

File: land_description/urdf/land_description.urdf (robot description, URDF)
Before this commit: robot land, 6 links, 5 joints
Joints:
- joint imu_joint: origin xyz=${0.01+tower_length/2} 0 ${base_height/2} rpy=0 0 0 -> xyz=${0.01+tower_length/2} 0 ${base_height/2} rpy=0 0 ${-pi/2}

File: land_description/urdf/land_description.urdf.xacro (robot description, xacro)
@@ -200,5 +200,5 @@
     <parent link="base_link"/>
     <child link="imu_link"/>
-    <origin rpy="0 0 0" xyz="0.04 0 0.0305"/>
+    <origin rpy="0 0 -1.5707963267948966" xyz="0.04 0 0.0305"/>
   </joint>
   <!-- LIDAR -->

Commit message: revert urdf

File: land_description/urdf/land_description.urdf (robot description, URDF)
Before this commit: robot land, 6 links, 5 joints
Joints:
- joint imu_joint: origin xyz=${0.01+tower_length/2} 0 ${base_height/2} rpy=0 0 ${-pi/2} -> xyz=${0.01+tower_length/2} 0 ${base_height/2} rpy=0 0 0

File: land_description/urdf/land_description.urdf.xacro (robot description, xacro)
@@ -200,5 +200,5 @@
     <parent link="base_link"/>
     <child link="imu_link"/>
-    <origin rpy="0 0 -1.5707963267948966" xyz="0.04 0 0.0305"/>
+    <origin rpy="0 0 0" xyz="0.04 0 0.0305"/>
   </joint>
   <!-- LIDAR -->

Commit message: test

File: land_description/urdf/land_description.urdf (robot description, URDF)
Before this commit: robot land, 6 links, 5 joints
Joints:
- joint imu_joint: origin xyz=${0.01+tower_length/2} 0 ${base_height/2} rpy=0 0 0 -> xyz=${0.01+tower_length/2} 0 ${base_height/2} rpy=0 0 ${pi/2}

Commit message: revert urdf

File: land_description/urdf/land_description.urdf (robot description, URDF)
Before this commit: robot land, 6 links, 5 joints
Joints:
- joint imu_joint: origin xyz=${0.01+tower_length/2} 0 ${base_height/2} rpy=0 0 ${pi/2} -> xyz=${0.01+tower_length/2} 0 ${base_height/2} rpy=0 0 0

File: land_description/urdf/land_description.urdf.xacro (robot description, xacro)
@@ -200,5 +200,5 @@
     <parent link="base_link"/>
     <child link="imu_link"/>
-    <origin rpy="0 0 1.5707963267948966" xyz="0.04 0 0.0305"/>
+    <origin rpy="0 0 0" xyz="0.04 0 0.0305"/>
   </joint>
   <!-- LIDAR -->

Commit message: update imu_link transform

File: land_description/urdf/land_description.urdf (robot description, URDF)
Before this commit: robot land, 6 links, 5 joints
Links:
- link imu_link: geometry collision box size=0.01 0.02 0.001; visual box size=0.01 0.02 0.001
Joints:
- joint imu_joint: origin xyz=${0.01+tower_length/2} 0 ${base_height/2} rpy=0 0 0 -> xyz=${0.01+tower_length/2} 0 ${base_height/2} rpy=0 0 ${-pi/2}

File: land_description/urdf/land_description.urdf.xacro (robot description, xacro)
@@ -179,5 +179,5 @@
       <origin rpy="0 0 0" xyz="0 0 0"/>
       <geometry>
-        <box size="0.02 0.01 0.001"/>
+        <box size="0.01 0.02 0.001"/>
       </geometry>
     </collision>
@@ -185,10 +185,10 @@
       <origin rpy="1.5707963267948966 0 1.5707963267948966" xyz="0 0 0"/>
       <mass value="0.01"/>
-      <inertia ixx="8.416666666666667e-08" ixy="0.0" ixz="0.0" iyy="4.166666666666667e-07" iyz="0.0" izz="3.341666666666667e-07"/>
+      <inertia ixx="3.341666666666667e-07" ixy="0.0" ixz="0.0" iyy="4.166666666666667e-07" iyz="0.0" izz="8.416666666666667e-08"/>
     </inertial>
     <visual>
       <origin rpy="0 0 0" xyz="0 0 0"/>
       <geometry>
-        <box size="0.02 0.01 0.001"/>
+        <box size="0.01 0.02 0.001"/>
       </geometry>
       <material name="Cyan">
@@ -200,5 +200,5 @@
     <parent link="base_link"/>
     <child link="imu_link"/>
-    <origin rpy="0 0 0" xyz="0.04 0 0.0305"/>
+    <origin rpy="0 0 -1.5707963267948966" xyz="0.04 0 0.0305"/>
   </joint>
   <!-- LIDAR -->

Commit message: update imu_link transform

File: land_description/urdf/land_description.urdf (robot description, URDF)
Before this commit: robot land, 6 links, 5 joints
Joints:
- joint imu_joint: origin xyz=${0.01+tower_length/2} 0 ${base_height/2} rpy=0 0 ${-pi/2} -> xyz=${0.01+tower_length/2} 0 ${base_height/2} rpy=0 0 ${pi/2}

File: land_description/urdf/land_description.urdf.xacro (robot description, xacro)
@@ -200,5 +200,5 @@
     <parent link="base_link"/>
     <child link="imu_link"/>
-    <origin rpy="0 0 -1.5707963267948966" xyz="0.04 0 0.0305"/>
+    <origin rpy="0 0 1.5707963267948966" xyz="0.04 0 0.0305"/>
   </joint>
   <!-- LIDAR -->

Commit message: increase ekf frequency

File: land_description/urdf/land_description.urdf (robot description, URDF)
Before this commit: robot land, 6 links, 5 joints
Links:
- link imu_link: geometry collision box size=0.02 0.01 0.001; visual box size=0.01 0.02 0.001

File: land_description/urdf/land_description.urdf.xacro (robot description, xacro)
@@ -179,5 +179,5 @@
       <origin rpy="0 0 0" xyz="0 0 0"/>
       <geometry>
-        <box size="0.01 0.02 0.001"/>
+        <box size="0.02 0.01 0.001"/>
       </geometry>
     </collision>
